File: PCB/Audio/Audio.kicad_pcb (KiCad board)
At the start: 2 copper layers, 70 x 70 mm, 35 parts, among them J1 Reset, J2 Wago, J3 TC2030-USB-NL-DS, J5 USB-C-Socket-H, SW1 Button, U1 ICS43434_MEMS_Mic, U6 ESP32-S3-MINI-1, U7 MD8942

Commit message: Concept
Parts:
- removed D2: ~, RevK:DFN1006-2L
- removed J1: Reset, RevK:AA-Pad
- removed J2: Wago, RevK:WAGO-2060-453-998-404
- removed R1: 124K, RevK:R_0402
- removed R3: 10K, RevK:R_0402
- removed SW1: Button, RevK:SW_Push_1P1T_NO_6x6mm
- added C13: 100nF, RevK:C_0402, F.Cu at (89.0, 102.5)
- added J4: TF_PUSH, RevK:TF_PUSH, B.Cu at (98.5, 98.3)
- added U2: R, RevK:ICS43434_MEMS_Mic, F.Cu at (88.0, 105.7)
- U1: value ICS43434_MEMS_Mic -> L
- moved C8 33.9 mm to (87.0, 98.0), turned to 90 degrees
- moved C9 29.4 mm to (115.0, 94.0)
- moved U1 29.1 mm to (88.0, 94.3), turned to 90 degrees
- moved C7 28.0 mm to (117.5, 93.5)
- moved R2 27.6 mm to (115.0, 93.0)
- moved C6 7.57 mm to (88.5, 99.5), turned to -90 degrees
Connections:
- U6 pad 25: Net-(J1-Pin_2) -> unconnected-(U6-GPIO21-Pad25)
Routing:
- net DC: track 98.6 -> 0.00 mm, vias 7 -> 0
- net +3V3: track 76.1 -> 0.00 mm, vias 6 -> 0
- net D+: track 50.7 -> 0.00 mm, vias 2 -> 0
- net GND: track 47.5 -> 0.00 mm, vias 35 -> 0
- net D-: track 30.9 -> 0.00 mm, vias 2 -> 0
- net SCK: track 23.9 -> 0.00 mm, vias 2 -> 0
- net SD: track 20.2 -> 0.00 mm, vias 2 -> 0
- net Net-(U6-EN): track 20.1 -> 0.00 mm, vias 2 -> 0
- net WS: track 17.5 -> 0.00 mm, vias 2 -> 0
- net LED: track 14.9 -> 0.00 mm, vias 1 -> 0
- net BLINK: track 13.8 -> 0.00 mm
- net Net-(J1-Pin_2): track 12.9 -> 0.00 mm, vias 1 -> 0
- net Net-(J5-CC2): track 12.7 -> 0.00 mm, vias 2 -> 0
- net PUSH: track 12.0 -> 0.00 mm, vias 1 -> 0
- net ADC: track 11.5 -> 0.00 mm, vias 2 -> 0
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Other:
- board text removed: "Made by RevK www.me.uk"
