File: PCB/Audio/Audio.kicad_pcb (KiCad board)
At the start: 2 copper layers, 70 x 70 mm, 32 parts, among them J3 TC2030-USB-NL-DS, J4 TF_PUSH, J5 USB-C-Socket-H, U1 L, U2 R, U6 ESP32-S3-MINI-1, U7 MD8942

Commit message: Closer
Parts:
- removed C6: 10uF 35V, RevK:C_0603
- V2: moved to B.Cu
- moved C8 1.97 mm to (88.7, 97.0)
- moved J3 1.81 mm to (111.8, 105.1)
- moved C13 1.58 mm to (90.5, 103.0)
- moved C1 1.55 mm to (111.4, 105.3)
- moved C2 1.55 mm to (111.4, 102.0)
- moved C4 1.55 mm to (118.2, 106.9)
- moved R15 1.55 mm to (109.2, 92.6)
- moved C10 1.55 mm to (108.5, 95.8)
- moved C11 1.55 mm to (113.5, 95.8)
- moved C12 1.55 mm to (111.0, 96.5)
- moved C3 1.55 mm to (109.2, 101.9)
- moved C5 1.55 mm to (113.5, 102.7)
- moved C7 1.55 mm to (119.0, 93.5)
- moved C9 1.55 mm to (116.5, 94.0)
- moved D1 1.55 mm to (119.8, 106.4)
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
Commit message: Rework concept
Parts:
- removed C10: 10uF 35V, RevK:C_0603_
- removed C11: 10uF 6.3V, RevK:C_0603_
- removed C12: 100nF, RevK:C_0603_
- removed L2: 10uH, RevK:L_4x4_
- removed R14: 39k2, RevK:R_0402_
- removed R15: 1M, RevK:R_0402_
- removed R4: 124k, RevK:R_0402_
- removed U7: MD8942, RevK:SOT-23-6-MD8942
- added C16: 100uF, RevK:C_0805, F.Cu at (110.0, 93.0)
- added C6: 100nF, RevK:C_0402, F.Cu at (88.5, 100.0)
- added D2: ~, RevK:DFN1006-2L, F.Cu at (120.5, 93.0)
- added D3: MBR0530, RevK:D_SOD-123, F.Cu at (113.5, 98.3)
- added D4: ~, RevK:DFN1006-2L, B.Cu at (119.0, 106.5)
- added D5: XL-1010RGBC-WS2812B, RevK:SMD1010, F.Cu at (90.0, 100.0)
- added J1: JST-PH-SM4-TB, RevK:JST_PH_S2B-PH-SM4-TB_1x02-1MP_P2.00mm_Horizontal, B.Cu at (116.0, 97.0)
- added Q2: CJ2301, RevK:SOT-23, F.Cu at (113.5, 94.0)
- added R1: 10K, RevK:R_0402, F.Cu at (121.5, 94.5)
- added R8: 10K, RevK:R_0402, F.Cu at (118.5, 93.0)
- added SW1: SW_Push, RevK:TS-1092S-B3D2-G, B.Cu at (118.0, 103.5)
- added U3: TP4054, RevK:SOT-23-5, F.Cu at (109.9, 99.5)
- added U4: ME6211C33M5G-N, RevK:SOT-23-5, F.Cu at (109.9, 96.0)
- moved C7 1.00 mm to (119.0, 94.5)
Other:
- board text removed: "${CURRENT_DATE}"
- board text removed: "(5V WHEN USB)"
- board text removed: "+"
- board text removed: "-"
- board text removed: "11"
- board text removed: "21"
- board text removed: "3.3V I/O"
- board text removed: "35"
- board text removed: "4"
- board text removed: "4V-35V POWER"
- board text removed: "6"
- board text removed: "A"
- board text removed: "C42"
- board text removed: "D40"
- board text removed: "HomeIsWhereTheSmartIs"
- board text removed: "I2S"
- board text removed: "L"
- board text removed: "Made in China"
- board text removed: "U"
- board text removed: "W41"
- board text removed: "led.revk.uk"
- board text removed: "www.hiwtsi.uk"
- board text removed: "®"
- board text removed: "⎍"

Commit message: Initial tracking
Parts:
- removed C7: 10uF 35V, RevK:C_0603
- moved D2 12.8 mm to (109.0, 98.5), turned to -90 degrees
- moved R8 11.5 mm to (113.4, 103.3), turned to -90 degrees
- moved R1 9.11 mm to (112.5, 95.9), turned to 180 degrees
- moved Q2 7.20 mm to (111.8, 101.0), turned to 180 degrees
- moved D4 6.10 mm to (114.4, 102.5)
- moved D3 3.78 mm to (114.5, 94.7), turned to -90 degrees
- moved C2 2.73 mm to (108.9, 101.0), turned to 180 degrees
- moved U4 2.70 mm to (111.5, 93.9), turned to 180 degrees
- moved U3 2.35 mm to (111.6, 98.0)
- moved R2 1.85 mm to (118.4, 92.9)
- moved C16 1.55 mm to (108.7, 93.8), turned to 90 degrees
- moved C5 1.22 mm to (114.6, 103.1)
- moved C9 1.10 mm to (116.5, 92.9)
- moved J1 1.05 mm to (117.0, 97.0)
- moved SW1 0.50 mm to (118.5, 103.5)
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Connections:
- C16 pad 1: +3.3V -> +3V3
- C5 pad 1: DC -> VBUS
- J3 pad 1: DC -> VBUS
- J3 pad 2: DC -> VBUS
- J4 pad 4: SPWR -> +3V3
- J5 pad A4: DC -> VBUS
- J5 pad A9: DC -> VBUS
- J5 pad B4: DC -> VBUS
- J5 pad B9: DC -> VBUS
- U4 pad 5: +3.3V -> +3V3
- U6 pad 10: PUSH -> unconnected-(U6-GPIO6-Pad10)
- U6 pad 12: ADC -> unconnected-(U6-GPIO8-Pad12)
- U6 pad 15: unconnected-(U6-GPIO11-Pad15) -> SCK
- U6 pad 16: unconnected-(U6-GPIO12-Pad16) -> SDSS
- U6 pad 17: unconnected-(U6-GPIO13-Pad17) -> SDMOSI
- U6 pad 19: unconnected-(U6-GPIO15-Pad19) -> SDSCK
- U6 pad 20: unconnected-(U6-GPIO16-Pad20) -> SDMISO
- U6 pad 21: unconnected-(U6-GPIO17-Pad21) -> SDCD
- U6 pad 33: unconnected-(U6-GPIO37-Pad33) -> BUTTON
- U6 pad 36: SD -> unconnected-(U6-GPIO40-Pad36)
- U6 pad 37: WS -> unconnected-(U6-GPIO41-Pad37)
- U6 pad 38: SCK -> unconnected-(U6-GPIO42-Pad38)
- U6 pad 4: unconnected-(U6-GPIO0-Pad4) -> WS
- U6 pad 40: unconnected-(U6-GPIO44-Pad40) -> CHARGING
- U6 pad 5: unconnected-(U6-GPIO1-Pad5) -> SD
- U6 pad 7: unconnected-(U6-GPIO3-Pad7) -> BLINK2
- U6 pad 8: LED -> unconnected-(U6-GPIO4-Pad8)
Routing:
- net +3V3: track 0.00 -> 94.8 mm, vias 0 -> 8
- net GND: track 0.00 -> 55.6 mm, vias 0 -> 9
- net D-: track 0.00 -> 37.7 mm, vias 0 -> 2
- net D+: track 0.00 -> 37.0 mm, vias 0 -> 2
- net VBUS: track 0.00 -> 19.8 mm, vias 0 -> 1
- net SCK: track 0.00 -> 18.1 mm, vias 0 -> 2
- net Net-(J5-CC2): track 0.00 -> 17.9 mm, vias 0 -> 2
- net SDCD: track 0.00 -> 17.8 mm, vias 0 -> 1
- net SDMISO: track 0.00 -> 16.9 mm, vias 0 -> 1
- net SDSCK: track 0.00 -> 16.8 mm, vias 0 -> 1
- net SDMOSI: track 0.00 -> 16.1 mm, vias 0 -> 1
- net SDSS: track 0.00 -> 16.0 mm, vias 0 -> 1
- net BLINK: track 0.00 -> 15.0 mm, vias 0 -> 2
- net SD: track 0.00 -> 13.6 mm, vias 0 -> 2
- net WS: track 0.00 -> 13.2 mm, vias 0 -> 2
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
Commit message: Position
Parts:
- moved J4 2.45 mm to (100.0, 100.8)

Commit message: Tidy tracks
Routing:
- net +3V3: track 94.8 -> 100.7 mm
- net Net-(D3-K): track 11.9 -> 13.7 mm
- net D+: track 37.0 -> 38.7 mm
- net BLINK: track 15.0 -> 16.3 mm
- net D-: track 37.7 -> 36.6 mm
- net VBUS: track 19.8 -> 19.2 mm
- net GND: vias 9 -> 18
Other:
- board text added: "${CURRENT_DATE}"

Commit message: Tidy
Parts:
- removed C5: 10uF 35V, RevK:C_0603
- added C11: 10uF 6.3V, RevK:C_0402, F.Cu at (114.4, 103.3)
- added C7: 10uF 6.3V, RevK:C_0402, B.Cu at (112.8, 97.0)
- U1: value L -> R
- U2: value R -> L
- moved R1 0.40 mm to (112.9, 95.9)
- moved U2 0.30 mm to (89.5, 106.0)
- moved U1 0.28 mm to (89.5, 94.0)
- moved U3 0.06 mm to (111.6, 97.9)
Connections:
- U1 pad 2: GND -> +3V3
- U2 pad 2: +3V3 -> GND
Routing:
- net GND: track 55.6 -> 64.8 mm, vias 18 -> 22
- net +3V3: track 100.7 -> 97.9 mm
- net Net-(D3-K): track 13.7 -> 11.8 mm
- net SD: track 13.6 -> 14.1 mm
- net WS: track 13.2 -> 12.6 mm
- added copper zone on F.Cu, net Net-(D3-K)
- added copper zone on F.Cu, net VBUS
Other:
- board text added: "A"
- board text added: "Audio"
- board text added: "L"
- board text added: "R"
- board text added: "audio.revk.uk"
