File: PCB/Audio/Audio.kicad_sch (KiCad schematic)
At the start: 34 parts, among them J1 Reset, J2 Wago, J3 TC2030-USB-NL-DS, J5 USB-C-Socket-H, SW1 Button, U1 ICS43434_MEMS_Mic, U2 ESP32-S3-MINI-1, U5 MD8942

Commit message: Concept
Parts:
- removed D2: ~, RevK:DFN1006-2L, symbol RevK:ES05D1MC10
- removed J1: Reset, RevK:AA-Pad, symbol Connector_Generic:Conn_01x02
- removed J2: Wago, RevK:WAGO-2060-453-998-404, symbol Connector_Generic:Conn_01x03
- removed R1: 124K, RevK:R_0402, symbol Device:R
- removed R3: 10K, RevK:R_0402, symbol Device:R
- removed SW1: Button, RevK:SW_Push_1P1T_NO_6x6mm, symbol Switch:SW_Push
- added C13: 100nF, RevK:C_0402, symbol Device:C
- added J4: TF_PUSH, RevK:TF_PUSH, symbol RevK:TF_PUSH
- added U2: R, RevK:ICS43434_MEMS_Mic, symbol RevK:ICS43434_MEMS_Mic
- U1: value ICS43434_MEMS_Mic -> L
Connections:
- net +3V3: now also C13.2, U2.2 (LR), U2.5 (VDD)
- net GND: now also C13.1, J4.6 (VSS), J4.S (SHIELD), U2.3 (GND)
- net SCK: now also U2.4 (SCK)
- net SD: now also U2.6 (SD)
- net WS: now also U2.1 (WS)
- new net SDCD: J4.9 (CD)
- new net SDMISO: J4.7 (DAT0)
- new net SDMOSI: J4.3 (CMD)
- new net SDSCK: J4.5 (CLK)
- new net SDSS: J4.2 (DAT3/CD)
- new net SPWR: J4.4 (VDD)
- no-connect marks 30 -> 32
Other:
- title: LED driver -> Audio
- moved on the sheet: C4, D4, J3
