File: PCB/Audio/Audio.kicad_sch (KiCad schematic)
At the start: 41 parts, among them J1 Battery, J3 TC2030-USB-NL-DS, J4 TF_PUSH, J5 USB-C-Socket-H, Q2 CJ2301, SW1 SW_Push, U1 R, U2 ESP32-S3-MINI-1, U2 L, U3 TP4054, U4 ME6211C33M5G-N

Commit message: Reworked
Connections:
- net BLINK2: now also U2.13 (GPIO9); no longer U2.7 (GPIO3)
- net BUTTON: now also U2.5 (GPIO1); no longer U2.8 (GPIO4)
- net CHARGING: now also U2.22 (GPIO18)
- net GND: now also U2.12 (GPIO8), U2.15 (GPIO11), U2.6 (GPIO2)
- net SCK: now also U2.14 (GPIO10); no longer U2.15 (GPIO11)
- net SD: now also U2.11 (GPIO7); no longer U2.5 (GPIO1)
- net WS: now also U2.10 (GPIO6); no longer U2.9 (GPIO5)
- no-connect marks 26 -> 22

Commit message: New layout
Parts:
- removed D4: ~, RevK:DFN1006-2L, symbol RevK:ES05D1MC10
- added C10, C5: 100nF, RevK:C_0402, symbol Device:C
- added D4, D6: XL-1010RGBC-WS2812B, RevK:SMD1010, symbol RevK:WS2812B-1mm
- added J2: Reset, RevK:AA-Pad, symbol Connector_Generic:Conn_01x02
- added R3: 10K, RevK:R_0402, symbol Device:R
Connections:
- net +3V3: now also C10.1, C5.1, D4.2 (+), D6.2 (+), R3.1
- net CHARGING: no longer U2.40 (GPIO44)
- net GND: now also J1.2 (Pin_2), C10.2, C5.2, D4.3 (-), D6.3 (-), J2.1 (Pin_1); no longer J1.1 (Pin_1), U2.12 (GPIO8), U2.15 (GPIO11), U2.6 (GPIO2)
- net SDCD: now also R3.2
- net SDMISO: now also U2.19 (GPIO15); no longer U2.20 (GPIO16)
- net SDSCK: now also U2.18 (GPIO14); no longer U2.19 (GPIO15)
- net VBAT: now also J1.1 (Pin_1); no longer J1.2 (Pin_2)
- net SDDAT1: now reaches J4.8 (DAT1), R9.2
- net SDDAT1: now also U2.20 (GPIO16)
- net at U2.25 (GPIO21): now also J2.2 (Pin_2)
- net at D5.1 (O): now also D4.4 (I)
- net at D4.1 (O): now also D6.4 (I)
- no-connect marks 22 -> 24
Other:
- moved on the sheet: C1, C11, C2, C3, C4, C6, C7, D4, D5
