File: PCB/Intercom/Intercom.kicad_sch (KiCad schematic)
At the start: 33 parts, among them J1 Reset, J2 Battery, J3 TC2030-USB-NL-DS, J5 USB-C-Socket-H, Q1 CJ2301, SW2 SW_Push, U2 ESP32-S3-MINI-1, U2 MAX98357A, U3 TP4054, U4 ME6211C33M5G-N, U5 L, U7 R

Commit message: Tidy SS
Other:
- title: LED driver -> Intercom
Changed lines of the file:
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@@
 	(paper "A4")
 	(title_block
-		(title "LED driver")
+		(title "Intercom")
 		(rev "1")
 		(comment 1 "@TheRealRevK")
