File: PCB/OSC/OCS.kicad_sch (KiCad schematic)
At the start: 42 parts, among them J1 Reset, J2 Wago, J3 TC2030-USB-NL-DS, J4 DC, J5 USB-C-Socket-H, J6 RELAY1, J7 RELAY2, SW1 Button, SW2 SW_Reed, U1 ICS43434_MEMS_Mic, U2 ESP32-S3-MINI-1, U3 Relay, U4 78L05, U5 MD8942, U8 Relay, U9 VEML6040

Commit message: Tracked
Parts:
- SW2: footprint (none) -> RevK:Reed-59170; LCSC Part # (none) -> C315909
Connections:
- net +3.3V is gone; now on net +3V3: U9.4 (VDD)
- net PUSH2: now also U2.22 (GPIO18)
- net RELAY2: now also U2.21 (GPIO17)
- net SCL: now also U2.19 (GPIO15)
- net SDA: now also U2.18 (GPIO14)
- net PUSH1: now reaches U2.20 (GPIO16)
- net PUSH1: now also D3.2, SW1.1
- net IR: no longer names the net of U2.30 (GPIO48)
- removed net PUSH: D3.2, SW1.1, U2.15 (GPIO11)
- net SKPPWR: no longer names the net of U2.40 (GPIO44)
- net SKPSCK: no longer names the net of U2.6 (GPIO2)
- net SKPSD: no longer names the net of U2.7 (GPIO3)
- net SKPWS: no longer names the net of U2.5 (GPIO1)
- no-connect marks 24 -> 25
Other:
- moved on the sheet: D5, SW2

Commit message: New layout
Connections:
- net PUSH1 renamed PUSH
- net PUSH2 renamed REED
Changed lines of the file:
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@@
 		)
 	)
-	(global_label "PUSH2"
+	(global_label "REED"
 		(shape output)
 		(at 197.485 114.3 180)
@@
 		)
 		(property "Intersheetrefs" "${INTERSHEET_REFS}"
-			(at 188.804 114.3 0)
+			(at 190.316 114.3 0)
 			(effects
 				(font
@@
 		)
 	)
-	(global_label "PUSH1"
+	(global_label "PUSH"
 		(shape input)
 		(at 35.56 88.9 180)
@@
 		)
 		(property "Intersheetrefs" "${INTERSHEET_REFS}"
-			(at 26.879 88.9 0)
+			(at 28.0885 88.9 0)
 			(effects
 				(font
@@
 		)
 	)
-	(global_label "PUSH1"
+	(global_label "PUSH"
 		(shape output)
 		(at 163.83 114.3 180)
@@
 		)
 		(property "Intersheetrefs" "${INTERSHEET_REFS}"
-			(at 155.149 114.3 0)
-			(effects
-				(font
-					(size 1.27 1.27)
-				)
-				(justify right)
-				(hide yes)
-			)
-		)
-	)
-	(global_label "PUSH2"
+			(at 156.3585 114.3 0)
+			(effects
+				(font
+					(size 1.27 1.27)
+				)
+				(justify right)
+				(hide yes)
+			)
+		)
+	)
+	(global_label "REED"
 		(shape input)
 		(at 35.56 93.98 180)
@@
 		)
 		(property "Intersheetrefs" "${INTERSHEET_REFS}"
-			(at 26.879 93.98 0)
-			(effects
-				(font
+			(at 28.391 93.98 0)
+			(effects
+				(font

Commit message: Ready to order
Parts:
- added D4: ~, RevK:DFN1006-2L, symbol RevK:ES05D1MC10
- added SW3: SW_Push, RevK:TS-1092S-B3D2-G, symbol Switch:SW_Push
- SW1: value Button -> SW_Push; footprint RevK:SW_Push_1P1T_NO_6x6mm -> RevK:TS-1092S-B3D2-G; now in the parts list
Connections:
- net GND: now also SW1.1, D4.1, SW3.1; no longer SW1.2
- net PUSH1: now reaches U2.31 (GPIO35)
- net PUSH1: now also D3.2, SW3.2
- net PUSH2: now reaches U2.32 (GPIO36)
- net PUSH2: now also SW1.2, D4.2
- removed net PUSH: D3.2, SW1.1, U2.20 (GPIO16)
- no-connect marks 25 -> 24
