File: PCB/OSC/OCS.kicad_pcb (KiCad board)
At the start: 2 copper layers, 46 x 33 mm, 42 parts, among them J1 Reset, J2 Wago, J3 TC2030-USB-NL-DS, J4 DC, J5 USB-C-Socket-H, J6 RELAY1, J7 RELAY2, SW1 Button, U1 ICS43434_MEMS_Mic, U3 Relay, U4 78L05, U6 ESP32-S3-MINI-1, U7 MD8942, U8 Relay, U9 VEML6040

Commit message: Tracked
Parts:
- added SW2: SW_Reed, RevK:Reed-59170, F.Cu at (106.0, 113.5)
- moved D3 30.0 mm to (113.2, 108.5), turned to -90 degrees
- moved R10 19.3 mm to (95.5, 105.5)
- moved C1 18.2 mm to (99.5, 107.5), turned to 90 degrees
- moved D5 16.0 mm to (97.4, 111.5)
- moved R5 7.93 mm to (113.1, 104.0)
- moved R6 7.93 mm to (114.0, 104.0)
- moved SW1 4.72 mm to (107.5, 107.5), turned to 180 degrees
- moved U9 3.16 mm to (120.0, 113.5)
- moved C8 3.00 mm to (113.0, 91.5), turned to 0 degrees
- moved J3 2.80 mm to (99.8, 107.4)
- moved U1 1.90 mm to (119.3, 92.5)
- moved U8 1.00 mm to (94.0, 110.5)
- moved R1 0.35 mm to (93.8, 104.6)
- moved R3 0.35 mm to (95.5, 104.6)
Connections:
- D3 pad 2: PUSH -> PUSH1
- SW1 pad 1: PUSH -> PUSH1
- U6 pad 15: PUSH -> unconnected-(U6-GPIO11-Pad15)
- U6 pad 18: unconnected-(U6-GPIO14-Pad18) -> SDA
- U6 pad 19: unconnected-(U6-GPIO15-Pad19) -> SCL
- U6 pad 20: unconnected-(U6-GPIO16-Pad20) -> PUSH1
- U6 pad 21: unconnected-(U6-GPIO17-Pad21) -> RELAY2
- U6 pad 22: unconnected-(U6-GPIO18-Pad22) -> PUSH2
- U6 pad 30: IR -> unconnected-(U6-GPIO48-Pad30)
- U6 pad 40: SKPPWR -> unconnected-(U6-GPIO44-Pad40)
- U6 pad 5: SKPWS -> unconnected-(U6-GPIO1-Pad5)
- U6 pad 6: SKPSCK -> unconnected-(U6-GPIO2-Pad6)
- U6 pad 7: SKPSD -> unconnected-(U6-GPIO3-Pad7)
- U9 pad 4: +3.3V -> +3V3
Routing:
- net GND: track 66.7 -> 18.9 mm, vias 40 -> 13
- net SCL: track 0.00 -> 40.4 mm, vias 0 -> 2
- net SDA: track 0.00 -> 35.3 mm, vias 0 -> 2
- net PUSH1: track 0.00 -> 34.6 mm, vias 0 -> 2
- net DC: track 134.7 -> 106.6 mm, vias 10 -> 3
- net SKPSD: track 26.4 -> 0.00 mm, vias 1 -> 0
- net SKPSCK: track 25.9 -> 0.00 mm, vias 1 -> 0
- net PUSH2: track 0.00 -> 23.7 mm, vias 0 -> 2
- net SKPWS: track 22.5 -> 0.00 mm, vias 2 -> 0
- net Net-(J7-Pin_2): track 0.00 -> 21.4 mm, vias 0 -> 2
- net SKPPWR: track 21.0 -> 0.00 mm, vias 2 -> 0
- net (no net): track 15.1 -> 0.00 mm
- net Net-(J7-Pin_1): track 0.00 -> 14.5 mm
- net D-: track 29.5 -> 42.9 mm
- net LED2: track 33.3 -> 22.2 mm, vias 2 -> 3
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Other:
- outline, holes or cut-outs redrawn
- board text added: "4 12 13 14 15 16 17 18 40 41 42"
- board text added: "Designed by RevK for RMLX Made in China"
- board text added: "LED RELAY1 ADC SDA SCL PUSH1 RELAY2 PUSH2 MICWS MICSD MICSCK"
- board text removed: "${CURRENT_DATE}"
- board text removed: "(5V WHEN USB)"
- board text removed: "+"
- board text removed: "-"
- board text removed: "11"
- board text removed: "12"
- board text removed: "13"
- board text removed: "3.3V I/O"
- board text removed: "4"
- board text removed: "44"
- board text removed: "48"
- board text removed: "4V-35V POWER"
- board text removed: "4Ω"
- board text removed: "6x6 BTN"
- board text removed: "A"
- board text removed: "ADC"
- board text removed: "C2"
- board text removed: "C42"
- board text removed: "D3"
- board text removed: "D41"
- board text removed: "HomeIsWhereTheSmartIs"
- board text removed: "I2S"
- board text removed: "IR 38kHz"
- board text removed: "L"
- board text removed: "L+R"
- board text removed: "Made in China"
- board text removed: "U"
- board text removed: "USB 5V"
- board text removed: "USB ONLY IF NOT EXTERFNAL POWER"
- board text removed: "W1"
- board text removed: "W40"
- board text removed: "led.revk.uk"
- board text removed: "www.hiwtsi.uk"
- board text removed: "®"
- board text removed: "⎍"

Commit message: New layout
Connections:
- net PUSH1 renamed PUSH
- net PUSH2 renamed REED
Other:
- board text added: "+"
- board text added: "-"
- board text added: "12"
- board text added: "13"
- board text added: "14 15"
- board text added: "16"
- board text added: "17"
- board text added: "18"
- board text added: "4"
- board text added: "40 41 42"
- board text added: "5V-35V ONLY WHEN NOT USB"
- board text added: "A"
- board text added: "ADC"
- board text added: "Designed by RevK for RMLX"
- board text added: "LED"
- board text added: "Made in China"
- board text added: "PUSH"
- board text added: "REED"
- board text added: "SDA SCL"
- board text added: "WS SD SCK"
- board text added: "⎍"
- board text removed: "4 12 13 14 15 16 17 18 40 41 42"
- board text removed: "Designed by RevK for RMLX Made in China"
- board text removed: "LED RELAY1 ADC SDA SCL PUSH1 RELAY2 PUSH2 MICWS MICSD MICSCK"

Commit message: Ready to order
Parts:
- added D4: ~, RevK:DFN1006-2L, F.Cu at (112.0, 110.0)
- added SW3: SW_Push, RevK:TS-1092S-B3D2-G, F.Cu at (118.0, 108.5)
- SW1: value Button -> SW_Push; footprint RevK:SW_Push_1P1T_NO_6x6mm -> RevK:TS-1092S-B3D2-G
- moved D3 1.66 mm to (114.0, 109.9), turned to 90 degrees
- moved SW1 1.12 mm to (108.0, 108.5), turned to 0 degrees
Connections:
- D3 pad 2: PUSH -> PUSH1
- SW1 pad 1: PUSH -> GND
- SW1 pad 2: GND -> PUSH2
- U6 pad 20: PUSH -> unconnected-(U6-GPIO16-Pad20)
- U6 pad 31: unconnected-(U6-GPIO35-Pad31) -> PUSH1
- U6 pad 32: unconnected-(U6-GPIO36-Pad32) -> PUSH2
Routing:
- net PUSH: track 34.6 -> 0.00 mm, vias 2 -> 0
- net PUSH1: track 0.00 -> 16.3 mm, vias 0 -> 2
- net PUSH2: track 0.00 -> 14.7 mm, vias 0 -> 2
- net GND: track 18.9 -> 23.9 mm, vias 13 -> 18
- net D-: track 42.9 -> 46.2 mm
- net DC: track 106.6 -> 103.9 mm
- net D+: track 29.1 -> 30.8 mm
- net REED: track 23.7 -> 23.0 mm
Other:
- board text added: "35"
- board text added: "36"
- board text added: "PUSH1"
- board text added: "PUSH2"
- board text removed: "16"
- board text removed: "PUSH"

Commit message: Moved LEDs
Other:
- board text added: "${CURRENT_DATE}"
