File: PCB/Recorder/Recorder.kicad_pcb (KiCad board)
At the start: 2 copper layers, 70 x 70 mm, 54 parts, among them J1 Battery, J2 Reset, J3 TC2030-USB-NL-DS, J4 TF_PUSH, J5 USB-C-Socket-H, Q2 CJ2301, SW1 SW_Push, U1 R, U2 L, U3 TP4054, U4 ME6211C33M5G-N, U5 MAX98357A, U6 ESP32-S3-MINI-1

Commit message: Tweak
Parts:
- moved J1 0.07 mm to (118.5, 105.0)
Routing:
- net Net-(D1-O): track 27.0 -> 26.4 mm

Commit message: Mdae longer
Routing:
- net GND: track 85.7 -> 71.2 mm
- net Net-(J5-CC1): track 15.5 -> 16.3 mm
- net VBAT: track 16.0 -> 16.7 mm
- net D-: track 37.3 -> 37.9 mm

Commit message: Hook
Parts:
- C12: renamed from C4; value 100nF -> 10uF
- C14: renamed from C12; value 10uF -> 100nF
- moved PCB1 5.00 mm to (95.0, 100.0)
- moved V1 5.00 mm to (95.0, 90.0)
- moved V2 5.00 mm to (95.0, 110.0)
- renumbered C14 to C4
Other:
- board text added: "41"
- board text removed: "37"

Commit message: Tidy
Parts:
- U1, U2: footprint RevK:ICS43434_MEMS_Mic -> RevK:ICS43434_MEMS_Mic_Open
- moved U1 2.59 mm to (89.0, 92.0), turned to 90 degrees
- moved U2 2.59 mm to (89.0, 108.0), turned to -90 degrees
Routing:
- net SCK: track 20.6 -> 37.2 mm, vias 1 -> 2
- net GND: track 71.2 -> 59.6 mm
- net BUTTON: track 23.4 -> 13.3 mm
- net WS: track 14.0 -> 21.5 mm, vias 2 -> 1
- net +3V3: track 128.7 -> 135.7 mm
- net SD: track 14.8 -> 20.7 mm
- net Net-(D4-I): track 27.0 -> 23.2 mm, vias 0 -> 2
- net Net-(U5-OUTN): track 6.23 -> 4.43 mm
Other:
- board text added: "AB"
- board text added: "QRQR"
